File: lets_split_panel/lets_split_panel.kicad_pcb (KiCad board)
At the start: 2 copper layers, 230.5 x 82 mm, 310 parts, among them J1 Speaker, J2 RST, J3 ISP, P1 WS2812>, P2 USB_OTG, P3 >WS2812, P4 Conn_01x04, SW1 MXALPS, SW1 SW_PUSH, SW10 MXALPS, SW10 SW_PUSH, SW11 MXALPS, SW11 SW_PUSH, SW12 MXALPS, SW12 SW_PUSH, SW13 MXALPS, SW13 SW_PUSH, SW14 MXALPS, SW14 SW_PUSH, SW15 MXALPS, SW15 SW_PUSH, SW16 MXALPS, SW16 SW_PUSH, SW17 MXALPS, SW17 SW_PUSH, SW18 MXALPS, SW18 SW_PUSH, SW19 MXALPS, SW19 SW_PUSH, SW2 MXALPS, SW2 SW_PUSH, SW20 MXALPS, SW20 SW_PUSH, SW21 MXALPS, SW21 SW_PUSH, SW22 MXALPS, SW22 SW_PUSH, SW23 MXALPS, SW23 SW_PUSH, SW24 MXALPS, SW24 SW_PUSH, SW3 MXALPS, SW3 SW_PUSH, SW4 MXALPS, SW4 SW_PUSH, SW5 MXALPS, SW5 SW_PUSH, SW6 MXALPS, SW6 SW_PUSH, SW7 MXALPS, SW7 SW_PUSH, SW8 MXALPS, SW8 SW_PUSH, SW9 MXALPS, SW9 SW_PUSH, U1 ATMega32U4, Y1 Crystal

Commit message: Finished panel
Parts:
- removed the C1 at (248.6, 64.4) (x2)
- removed the C1 at (132.3, 64.4)
- removed the C2 at (263.7, 68.6) (x2)
- removed the C2 at (147.5, 68.6)
- removed the C3 at (263.7, 65.3) (x2)
- removed the C3 at (147.5, 65.3)
- removed the C4 at (253.9, 60.4) (x2)
- removed the C4 at (137.7, 60.4)
- removed the D1 at (202.9, 81.4) (x2)
- removed the D1 at (86.6, 81.4) (x2)
- removed the D10 at (241.0, 100.5) (x2)
- removed the D10 at (124.7, 100.5) (x2)
- removed the D11 at (241.0, 119.5) (x2)
- removed the D11 at (124.7, 119.5) (x2)
- removed the D12 at (252.9, 133.2) (x2)
- removed the D12 at (136.7, 133.2) (x2)
- removed the D13 at (267.1, 81.4) (x2)
- removed the D13 at (150.9, 81.4) (x2)
- removed the D14 at (260.0, 100.5) (x2)
- removed the D14 at (143.8, 100.5) (x2)
- removed the D15 at (260.0, 119.5) (x2)
- removed the D15 at (143.8, 119.5) (x2)
- removed the D16 at (272.0, 133.2) (x2)
- removed the D16 at (155.7, 133.2) (x2)
- removed the D17 at (279.1, 81.4) (x2)
- removed the D17 at (162.8, 81.4) (x2)
- removed the D18 at (279.1, 100.5) (x2)
- removed the D18 at (162.8, 100.5) (x2)
- removed the D19 at (278.9, 119.5) (x2)
- removed the D19 at (162.7, 119.5) (x2)
- removed the D2 at (202.7, 100.5) (x2)
- removed the D2 at (86.5, 100.5) (x2)
- removed the D20 at (291.1, 133.2) (x2)
- removed the D20 at (174.9, 133.2) (x2)
- removed the D21 at (300.3, 81.4) (x2)
- removed the D21 at (184.0, 81.4) (x2)
- removed the D22 at (298.2, 100.5) (x2)
- removed the D22 at (182.0, 100.5) (x2)
- removed the D23 at (299.8, 119.5) (x2)
- removed the D23 at (183.5, 119.5) (x2)
- removed the D24 at (306.8, 133.2) (x2)
- removed the D24 at (190.5, 133.2) (x2)
- removed the D3 at (202.7, 119.5) (x2)
- removed the D3 at (86.5, 119.5) (x2)
- removed the D4 at (214.8, 133.2) (x2)
- removed the D4 at (98.6, 133.2) (x2)
- removed the D5 at (221.9, 81.4) (x2)
- removed the D5 at (105.7, 81.4) (x2)
- removed the D6 at (221.9, 100.5) (x2)
- removed the D6 at (105.7, 100.5) (x2)
- removed the D7 at (223.4, 119.5) (x2)
- removed the D7 at (107.2, 119.5) (x2)
- removed the D8 at (233.9, 133.2) (x2)
- removed the D8 at (117.6, 133.2) (x2)
- removed the D9 at (241.0, 81.4) (x2)
- removed the D9 at (124.7, 81.4) (x2)
- removed the J1 at (254.4, 82.3) (x2)
- removed the J1 at (138.2, 82.3)
- removed the J2 at (265.8, 61.5) (x2)
- removed the J2 at (149.5, 61.5)
- removed the J3 at (270.1, 65.3) (x2)
- removed the J3 at (153.9, 65.3)
- removed the JP1 at (272.4, 85.6) (x2)
- removed the JP1 at (156.1, 85.6)
- removed the JP2 at (274.8, 85.6) (x2)
- removed the JP2 at (158.6, 85.6)
- removed the P1 at (278.2, 62.6) (x2)
- removed the P1 at (161.9, 62.6)
- removed the P2 at (226.9, 60.0) (x2)
- removed the P2 at (110.7, 60.0)
- removed the P3 at (204.2, 68.7) (x2)
- removed the P3 at (88.0, 68.7)
- removed the P4 at (292.4, 64.9) (x2)
- removed the P4 at (176.2, 64.9)
- removed the R1 at (272.4, 89.9) (x2)
- removed the R1 at (156.1, 89.9)
- removed the R2 at (274.8, 89.9) (x2)
- removed the R2 at (158.6, 89.9)
- removed the R3 at (254.9, 76.2) (x2)
- removed the R3 at (138.7, 76.2)
- removed the R4 at (225.5, 67.9) (x2)
- removed the R4 at (109.2, 67.9)
- removed the R5 at (227.2, 67.9) (x2)
- removed the R5 at (111.0, 67.9)
- removed the R6 at (259.3, 61.7) (x2)
- removed the R6 at (143.1, 61.7)
- removed the REF** at (194.8, 104.0)
- removed the REF** at (194.8, 69.0)
- removed the REF** at (194.8, 72.0)
- removed the REF** at (197.6, 69.0)
- removed the REF** at (197.6, 72.0)
- removed the REF** at (197.6, 70.5)
- removed the REF** at (194.8, 70.5)
- removed the REF** at (194.8, 67.5)
- removed the REF** at (197.6, 131.1)
- removed the REF** at (197.6, 132.6)
- removed the REF** at (197.6, 134.1)
- removed the REF** at (197.6, 104.0)
- removed the REF** at (197.6, 135.6)
- removed the REF** at (194.8, 131.1)
- removed the REF** at (194.8, 132.6)
- removed the REF** at (194.8, 134.1)
- removed the REF** at (194.8, 135.6)
- removed the REF** at (216.2, 120.5) (x2)
- removed the REF** at (292.6, 120.5) (x2)
- removed the REF** at (292.4, 82.5) (x2)
- removed the REF** at (194.8, 99.5)
- removed the REF** at (176.3, 120.5)
- removed the REF** at (176.2, 82.5) (x2)
- removed the REF** at (100.0, 120.5)
- removed the REF** at (194.8, 102.5)
- removed the REF** at (197.6, 99.5)
- removed the REF** at (197.6, 102.5)
- removed the REF** at (197.6, 101.0)
- removed the REF** at (194.8, 101.0)
- removed the REF** at (197.6, 67.5)
- removed the SW1 at (206.8, 72.8)
- removed the SW1 at (90.5, 72.8)
- removed the SW10 at (263.9, 91.9) (x2)
- removed the SW10 at (147.7, 91.9)
- removed the SW11 at (282.9, 91.9) (x2)
- removed the SW11 at (166.7, 91.9)
- removed the SW12 at (302.0, 91.9) (x2)
- removed the SW12 at (185.8, 91.9)
- removed the SW13 at (206.8, 111.0) (x2)
- removed the SW13 at (90.5, 111.0)
- removed the SW14 at (225.8, 111.0) (x2)
- removed the SW14 at (109.5, 111.0)
- removed the SW15 at (244.8, 111.0) (x2)
- removed the SW15 at (128.6, 111.0)
- removed the SW16 at (263.9, 111.0) (x2)
- removed the SW16 at (147.7, 111.0)
- removed the SW17 at (282.9, 111.0) (x2)
- removed the SW17 at (166.7, 111.0)
- removed the SW18 at (302.0, 111.0) (x2)
- removed the SW18 at (185.8, 111.0)
- removed the SW19 at (206.8, 130.0) (x2)
- removed the SW19 at (90.5, 130.0)
- removed the SW2 at (225.8, 72.8) (x2)
- removed the SW2 at (109.5, 72.8)
- removed the SW20 at (225.8, 130.0) (x2)
- removed the SW20 at (109.5, 130.0)
- removed the SW21 at (244.8, 130.0) (x2)
- removed the SW21 at (128.6, 130.0)
- removed the SW22 at (263.9, 130.0) (x2)
- removed the SW22 at (147.7, 130.0)
- removed the SW23 at (282.9, 130.0) (x2)
- removed the SW23 at (166.7, 130.0)
- removed the SW24 at (302.0, 130.0) (x2)
- removed the SW24 at (185.8, 130.0)
- removed the SW3 at (244.8, 72.8) (x2)
- removed the SW3 at (128.6, 72.8) (x2)
- removed the SW4 at (263.9, 72.8) (x2)
- removed the SW4 at (147.7, 72.8)
- removed the SW5 at (282.9, 72.8) (x2)
- removed the SW5 at (166.7, 72.8)
- removed the SW6 at (302.0, 72.8) (x2)
- removed the SW7 at (206.8, 91.9) (x2)
- removed the SW7 at (90.5, 91.9)
- removed the SW8 at (225.8, 91.9) (x2)
- removed the SW8 at (109.5, 91.9)
- removed the SW9 at (244.8, 91.9) (x2)
- removed the SW9 at (128.6, 91.9)
- removed the U1 at (254.3, 67.2) (x2)
- removed the U1 at (138.1, 67.2)
- removed the Y1 at (261.6, 66.9) (x2)
- removed the Y1 at (145.3, 66.9) (x2)
- added C5: 1uF, SeeedOPL-Capacitor-2016:C0603, B.Cu at (172.4, 64.6)
- added C6: 8pF, SeeedOPL-Capacitor-2016:C0402, B.Cu at (187.5, 68.8)
- added C7: 8pF, SeeedOPL-Capacitor-2016:C0402, B.Cu at (187.5, 65.5)
- added C8: 1uF, SeeedOPL-Capacitor-2016:C0603, B.Cu at (177.7, 60.6)
- added D1: D, SeeedOPL-Diode-2016:SOD-123, B.Cu at (29.6, 81.4)
- added D10: D, SeeedOPL-Diode-2016:SOD-123, B.Cu at (67.7, 100.5)
- added D11: D, SeeedOPL-Diode-2016:SOD-123, B.Cu at (67.7, 119.5)
- added D12: D, SeeedOPL-Diode-2016:SOD-123, B.Cu at (79.7, 133.2)
- added D13: D, SeeedOPL-Diode-2016:SOD-123, B.Cu at (93.9, 81.4)
- added D14: D, SeeedOPL-Diode-2016:SOD-123, B.Cu at (86.8, 100.5)
- added D15: D, SeeedOPL-Diode-2016:SOD-123, B.Cu at (86.8, 119.5)
- added D16: D, SeeedOPL-Diode-2016:SOD-123, B.Cu at (98.7, 133.2)
- added D17: D, SeeedOPL-Diode-2016:SOD-123, B.Cu at (105.8, 81.4)
- added D18: D, SeeedOPL-Diode-2016:SOD-123, B.Cu at (105.8, 100.5)
- added D19: D, SeeedOPL-Diode-2016:SOD-123, B.Cu at (105.7, 119.5)
- added D2: D, SeeedOPL-Diode-2016:SOD-123, B.Cu at (29.5, 100.5)
- added D20: D, SeeedOPL-Diode-2016:SOD-123, B.Cu at (117.9, 133.2)
- added D21: D, SeeedOPL-Diode-2016:SOD-123, B.Cu at (127.0, 81.4)
- added D22: D, SeeedOPL-Diode-2016:SOD-123, B.Cu at (125.0, 100.5)
- added D23: D, SeeedOPL-Diode-2016:SOD-123, B.Cu at (126.5, 119.5)
- added D24: D, SeeedOPL-Diode-2016:SOD-123, B.Cu at (133.5, 133.2)
- added D25: D, SeeedOPL-Diode-2016:SOD-123, B.Cu at (150.0, 81.0)
- added D26: D, SeeedOPL-Diode-2016:SOD-123, B.Cu at (150.0, 100.0)
- added D27: D, SeeedOPL-Diode-2016:SOD-123, B.Cu at (149.5, 119.0)
- added D28: D, SeeedOPL-Diode-2016:SOD-123, B.Cu at (157.5, 135.0)
- added D29: D, SeeedOPL-Diode-2016:SOD-123, B.Cu at (169.0, 81.0)
- added D3: D, SeeedOPL-Diode-2016:SOD-123, B.Cu at (29.5, 119.5)
- added D30: D, SeeedOPL-Diode-2016:SOD-123, B.Cu at (169.0, 100.0)
- added D31: D, SeeedOPL-Diode-2016:SOD-123, B.Cu at (169.0, 119.0)
- added D32: D, SeeedOPL-Diode-2016:SOD-123, B.Cu at (176.5, 135.0)
- added D33: D, SeeedOPL-Diode-2016:SOD-123, B.Cu at (188.0, 81.0)
- added D34: D, SeeedOPL-Diode-2016:SOD-123, B.Cu at (188.0, 100.0)
- added D35: D, SeeedOPL-Diode-2016:SOD-123, B.Cu at (188.0, 119.0)
- added D36: D, SeeedOPL-Diode-2016:SOD-123, B.Cu at (195.5, 135.0)
- added D37: D, SeeedOPL-Diode-2016:SOD-123, B.Cu at (207.0, 81.0)
- added D38: D, SeeedOPL-Diode-2016:SOD-123, B.Cu at (207.0, 100.0)
- added D39: D, SeeedOPL-Diode-2016:SOD-123, B.Cu at (207.0, 119.0)
- added D4: D, SeeedOPL-Diode-2016:SOD-123, B.Cu at (41.6, 133.2)
- added D40: D, SeeedOPL-Diode-2016:SOD-123, B.Cu at (214.5, 135.0)
- added D41: D, SeeedOPL-Diode-2016:SOD-123, B.Cu at (226.5, 81.0)
- added D42: D, SeeedOPL-Diode-2016:SOD-123, B.Cu at (226.0, 100.0)
- added D43: D, SeeedOPL-Diode-2016:SOD-123, B.Cu at (226.0, 119.0)
- added D44: D, SeeedOPL-Diode-2016:SOD-123, B.Cu at (233.5, 135.0)
- added D45: D, SeeedOPL-Diode-2016:SOD-123, B.Cu at (245.0, 81.0)
- added D46: D, SeeedOPL-Diode-2016:SOD-123, B.Cu at (245.0, 100.0)
- added D47: D, SeeedOPL-Diode-2016:SOD-123, B.Cu at (245.0, 119.0)
- added D48: D, SeeedOPL-Diode-2016:SOD-123, B.Cu at (245.0, 135.0)
- added D5: D, SeeedOPL-Diode-2016:SOD-123, B.Cu at (48.7, 81.4)
- added D6: D, SeeedOPL-Diode-2016:SOD-123, B.Cu at (48.7, 100.5)
- added D7: D, SeeedOPL-Diode-2016:SOD-123, B.Cu at (50.2, 119.5)
- added D8: D, SeeedOPL-Diode-2016:SOD-123, B.Cu at (60.6, 133.2)
- added D9: D, SeeedOPL-Diode-2016:SOD-123, B.Cu at (67.7, 81.4)
- added J4: RST, Pin_Headers:Pin_Header_Straight_1x02_Pitch2.54mm, B.Cu at (189.6, 61.8)
- added J5: Speaker, Buzzers_Beepers:Buzzer_12x9.5RM7.6, B.Cu at (197.4, 82.3)
- added J6: ISP, Jlink:J-link-needle-6pin, B.Cu at (193.9, 65.5)
- added P5: USB_OTG, Connectors:USB-Mini-B-SMD, B.Cu at (224.8, 60.0)
- added P6: >WS2812, Wirepads:SMD_PAD_1x03_Pitch2.54mm, B.Cu at (172.7, 60.5)
- added P7: WS2812>, Wirepads:SMD_PAD_1x03_Pitch2.54mm, B.Cu at (149.5, 68.6)
- added P8: Conn_01x04, Connectors:SJ-4351X-SMT, B.Cu at (159.3, 64.9)
- added R10: 200, Resistors_SMD:R_0603_HandSoldering, B.Cu at (181.6, 83.9)
- added R7: 22R, Resistors_SMD:R_0603_HandSoldering, B.Cu at (205.0, 59.4)
- added R8: 22R, Resistors_SMD:R_0603_HandSoldering, B.Cu at (205.0, 61.0)
- added R9: 4k7, Resistors_SMD:R_0603_HandSoldering, B.Cu at (183.1, 62.0)
- added REF**: 1pin, Connect:1pin, F.Cu at (235.5, 120.5)
- added REF**: 1pin, Connect:1pin, F.Cu at (137.8, 103.5)
- added REF**: 1pin, Connect:1pin, F.Cu at (140.6, 102.0)
- added REF**: 1pin, Connect:1pin, F.Cu at (119.2, 82.5)
- added REF**: 1pin, Connect:1pin, F.Cu at (140.6, 132.1)
- added REF**: 1pin, Connect:1pin, F.Cu at (137.8, 133.6)
- added REF**: 1pin, Connect:1pin, F.Cu at (137.8, 130.6)
- added REF**: 1pin, Connect:1pin, F.Cu at (137.8, 132.1)
- added REF**: 1pin, Connect:1pin, F.Cu at (137.8, 135.1)
- added REF**: 1pin, Connect:1pin, F.Cu at (140.6, 130.6)
- added REF**: 1pin, Connect:1pin, F.Cu at (140.6, 135.1)
- added REF**: 1pin, Connect:1pin, F.Cu at (159.8, 120.5)
- added REF**: 1pin, Connect:1pin, F.Cu at (140.6, 133.6)
- added REF**: 1pin, Connect:1pin, F.Cu at (140.6, 71.0)
- added REF**: 1pin, Connect:1pin, F.Cu at (140.6, 68.0)
- added REF**: 1pin, Connect:1pin, F.Cu at (137.8, 68.0)
- added REF**: 1pin, Connect:1pin, F.Cu at (137.8, 72.5)
- added REF**: 1pin, Connect:1pin, F.Cu at (140.6, 72.5)
- added REF**: 1pin, Connect:1pin, F.Cu at (137.8, 71.0)
- added REF**: 1pin, Connect:1pin, F.Cu at (137.8, 69.5)
- added REF**: 1pin, Connect:1pin, F.Cu at (159.7, 82.5)
- added REF**: 1pin, Connect:1pin, F.Cu at (140.6, 69.5)
- added REF**: 1pin, Connect:1pin, F.Cu at (140.6, 100.5)
- added REF**: 1pin, Connect:1pin, F.Cu at (137.8, 100.5)
- added REF**: 1pin, Connect:1pin, F.Cu at (137.8, 102.0)
- added REF**: 1pin, Connect:1pin, F.Cu at (140.6, 103.5)
- added REF**: 1pin, Connect:1pin, F.Cu at (140.6, 99.0)
- added REF**: 1pin, Connect:1pin, F.Cu at (137.8, 99.0)
- added SW25: MXALPS, CherryMX:Kailh-socket, F.Cu at (149.8, 72.8)
- added SW26: MXALPS, CherryMX:Kailh-socket, F.Cu at (168.8, 72.8)
- added SW27: MXALPS, CherryMX:Kailh-socket, F.Cu at (187.8, 72.8)
- added SW28: MXALPS, CherryMX:Kailh-socket, F.Cu at (206.9, 72.8)
- added SW29: MXALPS, CherryMX:Kailh-socket, F.Cu at (225.9, 72.8)
- added SW3: MXALPS, CherryMX:Kailh-socket, F.Cu at (71.6, 72.8)
- added SW30: MXALPS, CherryMX:Kailh-socket, F.Cu at (245.0, 72.8)
- added SW31: MXALPS, CherryMX:Kailh-socket, F.Cu at (149.8, 91.9)
- added SW32: MXALPS, CherryMX:Kailh-socket, F.Cu at (168.8, 91.9)
- added SW33: MXALPS, CherryMX:Kailh-socket, F.Cu at (187.8, 91.9)
- added SW34: MXALPS, CherryMX:Kailh-socket, F.Cu at (206.9, 91.9)
- added SW35: MXALPS, CherryMX:Kailh-socket, F.Cu at (225.9, 91.9)
- added SW36: MXALPS, CherryMX:Kailh-socket, F.Cu at (245.0, 91.9)
- added SW37: MXALPS, CherryMX:Kailh-socket, F.Cu at (149.8, 111.0)
- added SW38: MXALPS, CherryMX:Kailh-socket, F.Cu at (168.8, 111.0)
- added SW39: MXALPS, CherryMX:Kailh-socket, F.Cu at (187.8, 111.0)
- added SW40: MXALPS, CherryMX:Kailh-socket, F.Cu at (206.9, 111.0)
- added SW41: MXALPS, CherryMX:Kailh-socket, F.Cu at (225.9, 111.0)
- added SW42: MXALPS, CherryMX:Kailh-socket, F.Cu at (245.0, 111.0)
- added SW43: MXALPS, CherryMX:Kailh-socket, F.Cu at (149.8, 130.0)
- added SW44: MXALPS, CherryMX:Kailh-socket, F.Cu at (168.8, 130.0)
- added SW45: MXALPS, CherryMX:Kailh-socket, F.Cu at (187.8, 130.0)
- added SW46: MXALPS, CherryMX:Kailh-socket, F.Cu at (206.9, 130.0)
- added SW47: MXALPS, CherryMX:Kailh-socket, F.Cu at (225.9, 130.0)
- added SW48: MXALPS, CherryMX:Kailh-socket, F.Cu at (245.0, 130.0)
- added U2: ATMega32U4, SeeedOPL-IC-2016:QFN44G-0.5-7X7MM, B.Cu at (178.1, 67.4)
- added Y1: Crystal, SeeedOPL-Crystal Oscillator-2016:X2-SMD-5.0X3.2X1.3MM, B.Cu at (88.3, 66.9)
- added Y2: Crystal, SeeedOPL-Crystal Oscillator-2016:X2-SMD-5.0X3.2X1.3MM, B.Cu at (185.4, 67.2)
- SW1, SW10, SW11, SW12, SW13, SW14, SW15, SW16, SW17, SW18, SW19, SW2, SW20, SW21, SW22, SW23, SW24, SW4, SW5, SW6, SW7, SW8, SW9: value SW_PUSH -> MXALPS
- moved JP2 57.0 mm to (101.6, 85.6)
- moved P1 57.0 mm to (104.9, 62.6)
- moved R2 57.0 mm to (101.6, 89.9)
- moved P2 57.0 mm to (53.6, 60.0)
- moved C1 57.0 mm to (75.3, 64.4)
- moved C2 57.0 mm to (90.5, 68.6)
- moved C3 57.0 mm to (90.5, 65.3)
- moved C4 57.0 mm to (80.7, 60.4)
- moved J3 57.0 mm to (96.9, 65.3)
- moved JP1 57.0 mm to (99.1, 85.6)
- moved P4 57.0 mm to (119.2, 64.9)
- moved R1 57.0 mm to (99.1, 89.9)
- moved R3 57.0 mm to (81.7, 76.2)
- moved REF** 57.0 mm to (43.0, 120.5)
- moved REF** 57.0 mm to (119.3, 120.5)
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Connections:
- net /D+ renamed /Left half/D+
- net /D- renamed /Left half/D-
- net MISO renamed /Left half/MISO
- net MOSI renamed /Left half/MOSI
- net Net-(P2-Pad2) renamed /Left half/Dd-
- net Net-(P2-Pad3) renamed /Left half/Dd+
- net SCK renamed /Left half/SCK
- net SCL/D3 renamed /Left half/SCL/D3
- net SDA renamed /Left half/SDA
- net WD2812-in renamed /Left half/wd2812-in
- net buzz renamed /Left half/buzz
- net col0 renamed /Left half/col0
- net col1 renamed /Left half/col1
- net col2 renamed /Left half/col2
- net col3 renamed /Left half/col3
- net col4 renamed /Left half/col4
- net col5 renamed /Left half/col5
- net ~RESET renamed /Left half/~Reset
- U1 pad 32: row2 -> /Left half/row2
- U1 pad 36: row3 -> /Left half/row3
- U1 pad 37: row1 -> /Left half/row1
- U1 pad 38: row0 -> /Left half/row0
Routing:
- net row3: track 821.9 -> 0.00 mm, vias 8 -> 0
- net row2: track 740.0 -> 0.00 mm, vias 8 -> 0
- net row1: track 666.5 -> 0.00 mm, vias 8 -> 0
- net row0: track 589.5 -> 0.00 mm
- net VBUS: track 864.1 -> 387.8 mm, vias 40 -> 19
- net /Left half/col5: track 546.7 -> 136.7 mm, vias 24 -> 6
- net GND: track 690.8 -> 358.2 mm, vias 38 -> 33
- net /Left half/col4: track 443.4 -> 110.9 mm, vias 20 -> 5
- net /Left half/col0: track 440.6 -> 110.1 mm, vias 24 -> 6
- net /Left half/col1: track 384.9 -> 96.2 mm, vias 20 -> 5
- net /Left half/SDA: track 357.0 -> 89.3 mm, vias 24 -> 6
- net /Left half/col3: track 355.6 -> 88.9 mm, vias 16 -> 4
- net /Left half/col2: track 291.3 -> 72.8 mm, vias 16 -> 4
- net /Left half/SCL/D3: track 285.4 -> 71.3 mm, vias 16 -> 4
- net /Left half/row3: track 0.00 -> 205.5 mm, vias 0 -> 2
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Other:
- outline, holes or cut-outs redrawn
- net class Default: trace_width 0.25 -> 0.1524
- board text added: "LET'S"
- board text added: "Let's Split, vitamins included by Duckle29"
- board text added: "SPLIT"
- board text removed: "LET'S SPLIT"
- board text removed: "Let's Split, vitamins included"
- board text removed: "by Duckle29"
