File: lets_split_panel/lets_split_panel.sch (KiCad schematic (older format))
At the start: 0 parts

Commit message: Added PnP files and split gerbers
Parts:
- added FID1, FID2, FID3, FID4, FID5, FID6: Fiducial, Fiducials:Fiducial_1mm_Dia_2mm_Outer, symbol fiducials:Fiducial
Changed lines of the file:
@@
 F1 "right.sch" 60
 $EndSheet
+$Comp
+L fiducials:Fiducial FID1
+U 1 1 5A2A708E
+P 3725 5125
+F 0 "FID1" H 3853 5178 60  0000 L CNN
+F 1 "Fiducial" H 3853 5072 60  0000 L CNN
+F 2 "Fiducials:Fiducial_1mm_Dia_2mm_Outer" H 3725 5125 60  0001 C CNN
+F 3 "" H 3725 5125 60  0001 C CNN
+	1    3725 5125
+	1    0    0    -1
+$EndComp
+$Comp
+L fiducials:Fiducial FID2
+U 1 1 5A2A7142
+P 4700 5125
+F 0 "FID2" H 4828 5178 60  0000 L CNN
+F 1 "Fiducial" H 4828 5072 60  0000 L CNN
+F 2 "Fiducials:Fiducial_1mm_Dia_2mm_Outer" H 4700 5125 60  0001 C CNN
+F 3 "" H 4700 5125 60  0001 C CNN
+	1    4700 5125
+	1    0    0    -1
+$EndComp
+$Comp
+L fiducials:Fiducial FID3
+U 1 1 5A2A71BE
+P 6825 5075
+F 0 "FID3" H 6953 5128 60  0000 L CNN
+F 1 "Fiducial" H 6953 5022 60  0000 L CNN
+F 2 "Fiducials:Fiducial_1mm_Dia_2mm_Outer" H 6825 5075 60  0001 C CNN
+F 3 "" H 6825 5075 60  0001 C CNN
+	1    6825 5075
+	1    0    0    -1
+$EndComp
+$Comp
+L fiducials:Fiducial FID4
+U 1 1 5A2A7248
+P 7800 5075
+F 0 "FID4" H 7928 5128 60  0000 L CNN
+F 1 "Fiducial" H 7928 5022 60  0000 L CNN
+F 2 "Fiducials:Fiducial_1mm_Dia_2mm_Outer" H 7800 5075 60  0001 C CNN
+F 3 "" H 7800 5075 60  0001 C CNN
+	1    7800 5075
+	1    0    0    -1
+$EndComp
+$Comp
+L fiducials:Fiducial FID5
+U 1 1 5A2A77D2
+P 3725 5525
+F 0 "FID5" H 3853 5578 60  0000 L CNN
+F 1 "Fiducial" H 3853 5472 60  0000 L CNN
+F 2 "Fiducials:Fiducial_1mm_Dia_2mm_Outer" H 3725 5525 60  0001 C CNN
+F 3 "" H 3725 5525 60  0001 C CNN
+	1    3725 5525
+	1    0    0    -1
+$EndComp
+$Comp
+L fiducials:Fiducial FID6
+U 1 1 5A2A7850
+P 6825 5525
+F 0 "FID6" H 6953 5578 60  0000 L CNN
+F 1 "Fiducial" H 6953 5472 60  0000 L CNN
+F 2 "Fiducials:Fiducial_1mm_Dia_2mm_Outer" H 6825 5525 60  0001 C CNN
+F 3 "" H 6825 5525 60  0001 C CNN
+	1    6825 5525
+	1    0    0    -1
+$EndComp
 $EndSCHEMATC

Commit message: Added kiwi
Parts:
- FID1, FID2, FID3, FID4, FID5, FID6: symbol fiducials:Fiducial -> lets_split_panel-rescue:Fiducial-RESCUE-lets_split_panel
Changed lines of the file:
@@
 $EndSheet
 $Comp
-L fiducials:Fiducial FID1
+L lets_split_panel-rescue:Fiducial-RESCUE-lets_split_panel FID1
 U 1 1 5A2A708E
 P 3725 5125
@@
 $EndComp
 $Comp
-L fiducials:Fiducial FID2
+L lets_split_panel-rescue:Fiducial-RESCUE-lets_split_panel FID2
 U 1 1 5A2A7142
 P 4700 5125
@@
 $EndComp
 $Comp
-L fiducials:Fiducial FID3
+L lets_split_panel-rescue:Fiducial-RESCUE-lets_split_panel FID3
 U 1 1 5A2A71BE
 P 6825 5075
@@
 $EndComp
 $Comp
-L fiducials:Fiducial FID4
+L lets_split_panel-rescue:Fiducial-RESCUE-lets_split_panel FID4
 U 1 1 5A2A7248
 P 7800 5075
@@
 $EndComp
 $Comp
-L fiducials:Fiducial FID5
+L lets_split_panel-rescue:Fiducial-RESCUE-lets_split_panel FID5
 U 1 1 5A2A77D2
 P 3725 5525
@@
 $EndComp
 $Comp
-L fiducials:Fiducial FID6
+L lets_split_panel-rescue:Fiducial-RESCUE-lets_split_panel FID6
 U 1 1 5A2A7850
 P 6825 5525
